File: PCBs/SB220.kicad_sch (KiCad schematic)
At the start: 93 parts, among them T1 HV Transformer, T2 Filament & Bias Transformer

Commit message: Completed standard SB-220 schematic page
Parts:
- removed C?: .02, symbol Device:C_Polarized_US
- removed L? (x2): L, symbol Device:L
- removed R? (x2): R_US, symbol Device:R_US
- removed SW? (x2): SW_SPST, symbol Switch:SW_SPST
- removed SW? (x2): SW_SPDT, symbol Switch:SW_SPDT
- removed SW?: SW_DP3T, symbol SB220:SW_Meter
- added C24, C51, C52, C53, C54: .02, symbol Device:C_Polarized_US
- added C29: .001 8kV, symbol Device:C_Polarized_US
- added C33, C34, C47: 22, symbol Device:C_Polarized_US
- added C35, C36: 115, symbol Device:C_Polarized_US
- added C37: 150, symbol Device:C_Polarized_US
- added C38: 180, symbol Device:C_Polarized_US
- added C39: 220, symbol Device:C_Polarized_US
- added C41, C44: 400, symbol Device:C_Polarized_US
- added C42, C45: 470, symbol Device:C_Polarized_US
- added C43, C46: 680, symbol Device:C_Polarized_US
- added C55: 250, symbol Device:C_Variable
- added C57: 437, symbol SB220:C_Variable_2x
- added D17: 56-26, symbol Device:D_Filled
- added D18: 56-24, symbol Device:D_Filled
- added J1: Ant Relay, symbol Connector:Conn_Coaxial
- added J2: ALC, symbol Connector:Conn_Coaxial
- added J3: RF Input, symbol Connector:Conn_Coaxial
- added J4: RF Output, symbol Connector:Conn_Coaxial
- added J5, J6: Screw_Terminal_01x04, symbol Connector:Screw_Terminal_01x04
- added K1: SB-220 Relay, symbol SB220:SB-220_Relay
- added L1: .58μH, symbol Device:L
- added L2: .6μH, symbol Device:L
- added L3: .93μH, symbol Device:L
- added L4: 1.65μH, symbol Device:L
- added L5: 2.95μH, symbol Device:L
- added L6: L_Variable, symbol SB220:L_Variable
- added L7: L_Variable, symbol SB220:L_Variable_2_Taps
- added PC1, PC2: Anode Cap, symbol SB220:3-500Z_Anode_Cap
- added R23: 47k, symbol Device:R_US
- added R24: 66k 1W, symbol Device:R_US
- added R25: 1k, symbol Device:R_US
- added R26: 100k, symbol Device:R_Potentiometer_US
- added R27: 100k, symbol Device:R_US
- added RFC-5: 45-4 1mH, symbol Device:L
- added RFC-6: 4.5-4 1mH, symbol Device:L
- added SW1: Power Switch, symbol SB220:SW_Power_Switch
- added SW2: SW_SPDT_2P, symbol SB220:SW_SPDT_2P
- added SW3: Bandswitch Wafer IR (From Rear), symbol SB220:Bandswitch
- added SW5: SW_Meter, symbol SB220:SW_Meter
- C1, C2: value C_Polarized_US -> .01 1.4kV
- C3, C5: renamed from C?; value C_Polarized_US -> .02
- C32: renamed from C?; value .02 -> .01 1.4kV
- C4: renamed from C?; value C_Polarized_US -> 20μF
- C48: renamed from C?; value .02 -> 10
- C49: renamed from C?; value .02 -> .001
- CB1, CB2: renamed from SW?; value SW_Push -> 10A
- D16: renamed from D?; value D_Filled -> 57-27
- M1: renamed from M?; value Fan -> Fan Motor
- P1: renamed from P?; value Conn_WallPlug_Earth -> 120/240 VAC 60Hz
- R1: renamed from R?; value R_US -> 1Ω 5W
- R2: renamed from R?; value R_US -> 3600Ω 5W
- R22: renamed from R?; value 33k -> 2.2k
- R3: renamed from R?; value R_US -> .82Ω 2W
- R6, R7, R8: renamed from R?; value R_US -> 4.7MΩ 1W
- R9: renamed from R?; value R_US -> 5.6kΩ
- RFC-1: renamed from L?; value L -> 45-61 50uH
- RFC-2: renamed from L?; value L -> 45-6 8.5uH
- RFC-3: renamed from T?; value Bifilar_Choke -> Bifilar_Choke 9μH
- RFC-4: renamed from L?; value L -> 45-4 1mH
- ZD1: renamed from D?; value D_Zener_Filled -> 5.1V
- gave numbers to parts that had none: 51
Connections:
- net GND is gone; now on net Earth: R3.2, R9.2
- net Earth: now also C24.2, C33.2, C34.2, C35.2, C36.2, C37.2, C38.2, C39.2, C41.2, C42.2, C43.2, C44.2, C45.2, C46.2, C51.2, C52.2, C53.2, C54.2, C55.2, C57.2, C57.2, J1.2 (Ext), J2.2 (Ext), J3.2 (Ext), J4.2 (Ext), R25.2, R26.3, RFC-5.2, RFC-6.2
- net at C5.1, MES2.2 (+): now also SW5.1
- net at C22.1, LA1.2 (+), LA2.2 (+)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: now also C24.1
- net at CB1.2: now also SW1.1 (A)
- net at M1.1 (+), T1.3 (BLK), T2.1 (BLK): now also SW1.2 (B)
- net at T1.7 (BLK/RED): now also SW2.4 (1)
- net at T2.4 (GRN/YEL): now also J7.2 (Pin_2), M1.2 (-), T2.2 (BLK/YEL), SW1.4 (B), SW2.2, SW2.5
- net at T1.8 (BLU): now also SW2.6
- net at R8.2, R9.1: now also SW5.4 (HV)
- net at C48.2, R11.1, R21.2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: now also D18.1 (K)
- net at CB2.2: now also SW1.3 (A)
- net at V2.CAP: now also PC2.2
- net at C21.1, RFC-3.1, V1.1: now also C32.1, V2.5; no longer V2.1
- net at C31.1, V2.2: now also RFC-5.1
- net at RFC-1.1: now also C29.1, PC1.1, PC2.1
- net at R1.2, R2.1, R3.1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: now also SW5.2 (GRID_MA)
- net at C48.1, R21.1: now also C47.2; no longer C32.2
- net at V1.CAP: now also PC1.2
- net at T1.4 (BLK/YEL): now also SW2.1
- net at T1.5 (YEL): now also SW2.3
- net at ZD1.1 (K): now also K1.5
- net at C21.2, RFC-3.3, V1.5: now also V2.1
- net at C4.1, D16.1 (K): now also K1.11, K1.2, R27.1
- new net: C54.1, D17.1 (K), R26.1
- new net: D17.2 (A), R24.2, R25.1
- new net: C35.1, L1.1, SW3.2 (10m)
- new net: C33.1, C34.1, L1.2, SW3.8 (10m)
- new net: C57.1, C57.1, K1.6, L7.4, RFC-6.1, SW3.6 (80m)
- new net: C36.1, L2.2, SW3.9 (15m)
- new net: C41.1, L4.2, SW3.11 (40m)
- new net: C38.1, L3.2, SW3.10 (20m)
- new net: C53.1, J2.1 (In), R23.2
- new net: K1.1, K1.3
- new net: J4.1 (In), K1.9, R24.1
- new net: C29.2, C55.1, L6.1
- new net: C39.1, L3.1, SW3.4 (20m)
- new net: C42.1, L4.1, SW3.5 (40m)
- new net: C51.1, D18.2 (A), R23.1
- new net: K1.6, R27.2
- new net: K1.6, T2.4 (GRN/YEL)
- new net: C43.1, C44.1, L5.2, SW3.12 (80m)
- new net: C37.1, L2.1, SW3.3 (15m)
- new net: C45.1, C46.1, L5.1, SW3.6 (80m)
- new net: J5.2 (Pin_2), J5.3 (Pin_3)
- new net: C52.1, J1.1 (In), K1.10
- new net: K1.4, SW3.1
- new net: C32.2, C47.1, SW3.7
- new net: J3.1 (In), K1.7
- new net: L6.3, L7.1, SW3.3 (15m)
- new net: L7.2, SW3.4 (20m)
- new net: L7.3, SW3.5 (40m)
- new net: L6.2, SW3.2 (10m)
- new net: J6.1 (Pin_1), J6.2 (Pin_2)
- new net: J6.3 (Pin_3), J6.4 (Pin_4)
- new net REL. PWR.: R26.2, SW5.3 (REL_PWR)
- no-connect marks 0 -> 2
Other:
- note added: "(Front)"
- note added: "(Off)"
- note added: "(SSB Position)"
- note added: "120VAC"
- note added: "240VAC"
- note added: "Bandswitch"
- note added: "Connections"
- note added: "Load"
- note added: "Meter"
- note added: "Mode Switch"
- note added: "Multi-"
- note added: "Notes: 1. All resistors are 1/2 watt unless otherwise indicated. Values are in ohms (1k = 1000, M = 1,000,000). 2. Capacitor values less than 1 are uF. Values of 1 and above are in pF unless otherwise indicated. 3. The bandswitch is in the 80 meter position. Arrows indicate the direction of rotation for the view shown."
- note added: "Power"
- note added: "Sensitivity"
- note added: "Strip"
- note added: "Switch"
- note added: "Terminal"
- note added: "Tune"
- moved on the sheet: C1, C10, C11, C12, C13, C14, C15, C16, C17, C19, C2, C21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

Commit message: Tweaked some things
Parts:
- K1: value Relay Coil -> SB-220 Relay
- renumbered C16 to C18, C5 to C8
Changed lines of the file:
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@@
     (stroke (width 0) (type default) (color 0 0 0 0))
   )
+  (polyline (pts (xy 469.9 95.885) (xy 497.205 139.065))
+    (stroke (width 0.4) (type default) (color 0 0 0 0))
+  )
   (wire (pts (xy 100.965 329.565) (xy 151.765 329.565))
     (stroke (width 0) (type default) (color 0 0 0 0))
@@
     (stroke (width 0) (type default) (color 0 0 0 0))
   )
+  (polyline (pts (xy 295.91 247.65) (xy 550.545 247.65))
+    (stroke (width 0) (type default) (color 0 0 0 0))
+  )
   (wire (pts (xy 456.565 345.44) (xy 474.345 345.44))
     (stroke (width 0) (type default) (color 0 0 0 0))
@@
     (stroke (width 0) (type default) (color 0 0 0 0))
   )
-  (polyline (pts (xy 273.685 261.62) (xy 287.02 261.62))
+  (polyline (pts (xy 273.685 263.525) (xy 287.02 263.525))
     (stroke (width 0.6) (type solid) (color 0 0 0 0))
   )
@@
     (stroke (width 0) (type default) (color 0 0 0 0))
   )
-  (polyline (pts (xy 287.02 261.62) (xy 287.02 252.73))
+  (polyline (pts (xy 287.02 263.525) (xy 287.02 254.635))
     (stroke (width 0.6) (type solid) (color 0 0 0 0))
   )
@@
     (stroke (width 0) (type default) (color 0 0 0 0))
   )
-  (polyline (pts (xy 287.02 252.73) (xy 273.685 252.73))
+  (polyline (pts (xy 287.02 254.635) (xy 273.685 254.635))
     (stroke (width 0.3) (type solid) (color 0 0 0 0))
   )
@@
     (stroke (width 0) (type default) (color 0 0 0 0))
   )
-  (wire (pts (xy 259.715 242.57) (xy 259.715 260.35))
+  (wire (pts (xy 257.175 242.57) (xy 257.175 260.35))
     (stroke (width 0) (type default) (color 0 0 0 0))
   )
@@
     (stroke (width 0) (type default) (color 0 0 0 0))
   )
-  (wire (pts (xy 259.715 260.35) (xy 219.075 260.35))
+  (wire (pts (xy 257.175 260.35) (xy 219.075 260.35))
     (stroke (width 0) (type default) (color 0 0 0 0))
   )
@@
     (stroke (width 0) (type default) (color 0 0 0 0))
   )
+  (polyline (pts (xy 270.51 253.365) (xy 295.91 247.65))
+    (stroke (width 0) (type default) (color 0 0 0 0))
+  )
   (wire (pts (xy 342.265 95.885) (xy 391.795 95.885))
     (stroke (width 0) (type default) (color 0 0 0 0))
@@
     (stroke (width 0) (type default) (color 0 0 0 0))
   )
-  (polyline (pts (xy 273.685 252.73) (xy 273.685 261.62))
+  (polyline (pts (xy 273.685 254.635) (xy 273.685 263.525))
     (stroke (width 0.3) (type solid) (color 0 0 0 0))
   )
@@
     (stroke (width 0) (type default) (color 0 0 0 0))
   )
-  (wire (pts (xy 266.7 242.57) (xy 259.715 242.57))
+  (wire (pts (xy 266.7 242.57) (xy 257.175 242.57))
     (stroke (width 0) (type default) (color 0 0 0 0))
   )
@@
     (effects (font (size 2.54 2.54) (thickness 0.508) bold) (justify left bottom))
   )
-  (text "Switch" (at 273.685 261.62 0)
+  (text "Switch" (at 273.685 263.525 0)
     (effects (font (size 2.54 2.54) (thickness 0.508) bold) (justify left bottom))
   )
@@
     (effects (font (size 1.27 1.27)) (justify right bottom))
   )
-  (text "Meter" (at 274.955 257.175 0)
+  (text "Meter" (at 274.955 259.08 0)
     (effects (font (size 2.54 2.54) (thickness 0.508) bold) (justify left bottom))
   )
@@
     (pin "4")
   )
-  (symbol (lib_id "SB220:SW_Meter") (at 559.435 253.365 0) (unit 2)
+  (symbol (lib_id "SB220:SW_Meter") (at 559.435 248.92 0) (unit 2)
     (in_bom yes) (on_board yes) (fields_autoplaced)
-    (property "Reference" "SW5" (id 0) (at 569.6139 252.2993 0)
+    (property "Reference" "SW5" (id 0) (at 569.6139 247.8543 0)
       (effects (font (size 1.27 1.27)) (justify left) hide)
     )
-    (property "Value" "SW_Meter" (id 1) (at 569.6138 253.6869 0)
+    (property "Value" "SW_Meter" (id 1) (at 569.6138 249.2419 0)
       (effects (font (size 1.27 1.27)) (justify left) hide)
     )
-    (property "Footprint" "" (id 2) (at 554.99 269.24 0)
+    (property "Footprint" "" (id 2) (at 554.99 264.795 0)
       (effects (font (size 1.27 1.27)) hide)
     )
-    (property "Datasheet" "~" (id 3) (at 554.99 269.24 0)
+    (property "Datasheet" "~" (id 3) (at 554.99 264.795 0)
       (effects (font (size 1.27 1.27)) hide)
     )
@@
       (effects (font (size 1.27 1.27)) (justify left))
     )
-    (property "Value" "Relay Coil" (id 1) (at 360.68 317.5 0)
+    (property "Value" "SB-220 Relay" (id 1) (at 360.68 317.5 0)
       (effects (font (size 1.27 1.27)) (justify left))
     )
@@
   (symbol (lib_id "Device:C_Polarized_US") (at 316.865 77.47 0) (unit 1)
     (in_bom yes) (on_board yes)
-    (property "Reference" "C16" (id 0) (at 313.69 75.9649 0)
+    (property "Reference" "C18" (id 0) (at 313.69 75.9649 0)
       (effects (font (size 1.27 1.27)) (justify right))
     )
@@
     (pin "2")
   )
-  (symbol (lib_id "SB220:SW_Meter") (at 270.51 250.19 0) (unit 1)
+  (symbol (lib_name "SW_Meter_1") (lib_id "SB220:SW_Meter") (at 270.51 250.19 0) (unit 1)
     (in_bom yes) (on_board yes) (fields_autoplaced)
     (property "Reference" "SW5" (id 0) (at 275.6662 254.1615 0)
@@
   (symbol (lib_id "Device:C_Polarized_US") (at 259.715 269.875 0) (unit 1)
     (in_bom yes) (on_board yes)
-    (property "Reference" "C5" (id 0) (at 256.54 267.97 0)
+    (property "Reference" "C8" (id 0) (at 256.54 267.97 0)
       (effects (font (size 1.27 1.27)) (justify right))
     )
@@
       (reference "C5") (unit 1) (value ".02") (footprint "")
     )
-    (path "/fa71034f-73d1-4013-a522-cd49212a34b2"
-      (reference "C5") (unit 1) (value ".02") (footprint "")
-    )
     (path "/06db77b5-089e-41f7-b42b-f6a395a0e131"
       (reference "C6") (unit 1) (value "200μF 450V") (footprint "")
@@
       (reference "C7") (unit 1) (value "200μF 450V") (footprint "")
     )
+    (path "/fa71034f-73d1-4013-a522-cd49212a34b2"
+      (reference "C8") (unit 1) (value ".02") (footprint "")
+    )
     (path "/f2590a7d-d6f0-4715-a043-4eb66b1de74d"
       (reference "C10") (unit 1) (value "200μF 450V") (footprint "")
@@
       (reference "C16") (unit 1) (value "200μF 450V") (footprint "")
     )
-    (path "/a7a1281e-7c4a-4d32-93a7-0f64240c7226"
-      (reference "C16") (unit 1) (value "200") (footprint "")
-    )
     (path "/303787e4-49f3-43a8-b3e8-6050266e165f"
       (reference "C17") (unit 1) (value "200μF 450V") (footprint "")
     )
+    (path "/a7a1281e-7c4a-4d32-93a7-0f64240c7226"
+      (reference "C18") (unit 1) (value "200") (footprint "")
+    )
     (path "/c1a9123d-a2ec-400e-9cf4-fbc88906c8e2"
       (reference "C19") (unit 1) (value "200") (footprint "")
@@
     )
     (path "/7e3035ff-10c0-4f0b-ae25-2f8486c4cb14"
-      (reference "K1") (unit 4) (value "Relay Coil") (footprint "")
+      (reference "K1") (unit 4) (value "SB-220 Relay") (footprint "")
     )
     (path "/02a6b2df-6b83-4670-9e03-78aa4897d274"
